Commit message: Feat: Add gz/moveit multi launch

File: config/frcobot_gz_moveit2.urdf.xacro (robot description, xacro)
@@ -1,14 +1,12 @@
-<!-- TODO: Try using launch args  -->
-<!-- The names of the MoveIt SRDF and the Gazebo Xacro don't match, which causes a lot of errors.
-It doesn't affect functionality, but it's unpleasant to see. -->
-<robot name="fairino_cobot" xmlns:xacro="http://www.ros.org/wiki/xacro">
-<!-- TODO: Try using launch args  -->
-<!-- TODO: If it's too difficult, create an additional xacro file. and retry  -->
+<?xml version="1.0"?>
+<robot name="$(arg robot_name)_robot" xmlns:xacro="http://www.ros.org/wiki/xacro">
   <xacro:arg name="robot_name" default="fairino5_v6"/>
+  <xacro:arg name="pkg_name_arg" default="fairino5_v6_moveit2_config"/>
   <xacro:property name="model" value="$(arg robot_name)"/>
+  <xacro:property name="pkg_name" value="$(arg robot_name)_moveit2_config"/>
   <xacro:include filename="$(find fairino_description)/urdf/${model}.urdf" />
   <xacro:include filename="$(find fairino_sim)/config/frcobot_gz_moveit2.xacro" />
   <xacro:include filename="$(find fairino_sim)/config/frcobot_gz_ros2_control.xacro" />
-  <xacro:frcobot_gz_moveit2 />
+  <xacro:frcobot_gz_moveit2 pkg_name="${pkg_name}" />
   <xacro:frcobot_gz_ros2_control />
 <!-- TODO: Later, configure it as a static tf node in the launch file.  -->

File: config/frcobot_gz_moveit2.xacro (robot description, xacro)
@@ -1,81 +1,81 @@
 <?xml version="1.0"?>
 <robot xmlns:xacro="http://www.ros.org/wiki/xacro">
-	<xacro:macro name="frcobot_gz_moveit2" params="namespace:=/">
-    <gazebo>
-      <plugin filename="gz_ros2_control-system" name="gz_ros2_control::GazeboSimROS2ControlPlugin">
-      <!-- TODO: Try using launch args ex)$(find args_name_descpition)config/${args yamlfile name}.yaml -->
-          <parameters>$(find fairino_sim)/config/frcobot_gz_moveit_controller2.yaml</parameters>
-        </plugin>
-    </gazebo>
-    <!-- Base -->
-    <gazebo reference="base_link">
-      <turnGravityOff>true</turnGravityOff>
-      <kp>0.0</kp>
-      <kd>0.0</kd>
-      <mu1>0.0</mu1>
-      <mu2>0.0</mu2>
-      <maxVel>0.0</maxVel>
-      <minDepth>0.0</minDepth>
-    </gazebo>
-    <!-- Link1 -->
-    <gazebo reference="shoulder_link">
-      <turnGravityOff>true</turnGravityOff>
-      <kp>0.0</kp>
-      <kd>0.0</kd>
-      <mu1>0.0</mu1>
-      <mu2>0.0</mu2>
-      <maxVel>0.0</maxVel>
-      <minDepth>0.0</minDepth>
-    </gazebo>
-    <!-- Link2 -->
-    <gazebo reference="upperarm_link">
-      <turnGravityOff>true</turnGravityOff>
-      <kp>0.0</kp>
-      <kd>0.0</kd>
-      <mu1>0.0</mu1>
-      <mu2>0.0</mu2>
-      <maxVel>0.0</maxVel>
-      <minDepth>0.0</minDepth>
-    </gazebo>
-    <!-- Link3 -->
-    <gazebo reference="forearm_link">
-      <turnGravityOff>true</turnGravityOff>
-      <kp>0.0</kp>
-      <kd>0.0</kd>
-      <mu1>0.0</mu1>
-      <mu2>0.0</mu2>
-      <maxVel>0.0</maxVel>
-      <minDepth>0.0</minDepth>
-    </gazebo>
-    <!-- Link4 -->
-    <gazebo reference="wrist1_link">
-      <turnGravityOff>true</turnGravityOff>
-      <kp>0.0</kp>
-      <kd>0.0</kd>
-      <mu1>0.0</mu1>
-      <mu2>0.0</mu2>
-      <maxVel>0.0</maxVel>
-      <minDepth>0.0</minDepth>
-    </gazebo>
-    <!-- Link5 -->
-    <gazebo reference="wrist2_link">
-      <turnGravityOff>true</turnGravityOff>
-      <kp>0.0</kp>
-      <kd>0.0</kd>
-      <mu1>0.0</mu1>
-      <mu2>0.0</mu2>
-      <maxVel>0.0</maxVel>
-      <minDepth>0.0</minDepth>
-    </gazebo>
-    <!-- Link6 -->
-    <gazebo reference="wrist3_link">
-      <turnGravityOff>true</turnGravityOff>
-      <kp>0.0</kp>
-      <kd>0.0</kd>
-      <mu1>0.0</mu1>
-      <mu2>0.0</mu2>
-      <maxVel>0.0</maxVel>
-      <minDepth>0.0</minDepth>
-    </gazebo>
-	</xacro:macro>
+  <xacro:macro name="frcobot_gz_moveit2" params="pkg_name">
+    <xacro:property name="pkg_arg" value="${pkg_name}"/>
+      <gazebo>
+        <plugin filename="gz_ros2_control-system" name="gz_ros2_control::GazeboSimROS2ControlPlugin">
+            <parameters>$(find ${pkg_arg})/config/ros2_controllers.yaml</parameters>
+          </plugin>
+      </gazebo>
+      <!-- Base -->
+      <gazebo reference="base_link">
+        <turnGravityOff>true</turnGravityOff>
+        <kp>0.0</kp>
+        <kd>0.0</kd>
+        <mu1>0.0</mu1>
+        <mu2>0.0</mu2>
+        <maxVel>0.0</maxVel>
+        <minDepth>0.0</minDepth>
+      </gazebo>
+      <!-- Link1 -->
+      <gazebo reference="shoulder_link">
+        <turnGravityOff>true</turnGravityOff>
+        <kp>0.0</kp>
+        <kd>0.0</kd>
+        <mu1>0.0</mu1>
+        <mu2>0.0</mu2>
+        <maxVel>0.0</maxVel>
+        <minDepth>0.0</minDepth>
+      </gazebo>
+      <!-- Link2 -->
+      <gazebo reference="upperarm_link">
+        <turnGravityOff>true</turnGravityOff>
+        <kp>0.0</kp>
+        <kd>0.0</kd>
+        <mu1>0.0</mu1>
+        <mu2>0.0</mu2>
+        <maxVel>0.0</maxVel>
+        <minDepth>0.0</minDepth>
+      </gazebo>
+      <!-- Link3 -->
+      <gazebo reference="forearm_link">
+        <turnGravityOff>true</turnGravityOff>
+        <kp>0.0</kp>
+        <kd>0.0</kd>
+        <mu1>0.0</mu1>
+        <mu2>0.0</mu2>
+        <maxVel>0.0</maxVel>
+        <minDepth>0.0</minDepth>
+      </gazebo>
+      <!-- Link4 -->
+      <gazebo reference="wrist1_link">
+        <turnGravityOff>true</turnGravityOff>
+        <kp>0.0</kp>
+        <kd>0.0</kd>
+        <mu1>0.0</mu1>
+        <mu2>0.0</mu2>
+        <maxVel>0.0</maxVel>
+        <minDepth>0.0</minDepth>
+      </gazebo>
+      <!-- Link5 -->
+      <gazebo reference="wrist2_link">
+        <turnGravityOff>true</turnGravityOff>
+        <kp>0.0</kp>
+        <kd>0.0</kd>
+        <mu1>0.0</mu1>
+        <mu2>0.0</mu2>
+        <maxVel>0.0</maxVel>
+        <minDepth>0.0</minDepth>
+      </gazebo>
+      <!-- Link6 -->
+      <gazebo reference="wrist3_link">
+        <turnGravityOff>true</turnGravityOff>
+        <kp>0.0</kp>
+        <kd>0.0</kd>
+        <mu1>0.0</mu1>
+        <mu2>0.0</mu2>
+        <maxVel>0.0</maxVel>
+        <minDepth>0.0</minDepth>
+      </gazebo>
+    </xacro:macro>
 </robot>
